Commit message: fix linke typo

File: riderless_bike_parameterized.urdf (robot description, URDF)
Before this commit: robot RiderlessBike, 12 links, 12 joints
Joints:
- joint floating_A_base_joint: child  -> floating_A_base

Commit message: remove disallowed prismatic joints

File: riderless_bike_parameterized.urdf (robot description, URDF)
Before this commit: robot RiderlessBike, 12 links, 12 joints
Links:
- removed link floating_A_base
- added link floating_x_base
- added link floating_y_base
Joints:
- removed joint floating_A_base_joint
- added joint floating_x_base_joint: type prismatic, parent world, child floating_x_base, axis 1 0 0
- added joint floating_y_base_joint: type prismatic, parent floating_x_base, child floating_y_base, axis 0 1 0
- joint floating_z_base_joint: parent floating_A_base -> floating_y_base

Commit message: remove __ typo

File: riderless_bike_parameterized.urdf (robot description, URDF)
Before this commit: robot RiderlessBike, 13 links, 13 joints
Joints:
- joint front_wheel_center_steer_basis_joint: child front_wheel__center_steer_basis -> front_wheel_center_steer_basis

Commit message: make wheels thinner

File: riderless_bike_parameterized.urdf (robot description, URDF)
Before this commit: robot RiderlessBike, 13 links, 13 joints
Links:
- link back_wheel: geometry visual cylinder length=.01 radius=${r_R}
- link front_wheel: geometry visual cylinder length=.01 radius=${r_F}
- link rear_frame: geometry visual cylinder length=${d1} radius=.02

Commit message: make front frame thinner

File: riderless_bike_parameterized.urdf (robot description, URDF)
Before this commit: robot RiderlessBike, 13 links, 13 joints
Links:
- link front_frame: geometry visual cylinder length=${d2} radius=.01

Commit message: ground smaller and at zero

File: riderless_bike_parameterized.urdf (robot description, URDF)
Before this commit: robot RiderlessBike, 13 links, 13 joints
Links:
- link ground: geometry visual box size=100 100 .05

Commit message: correct front wheel position

File: riderless_bike_parameterized.urdf (robot description, URDF)
Before this commit: robot RiderlessBike, 13 links, 13 joints
Joints:
- joint front_wheel_center_steer_basis_joint: origin xyz=${-L3} 0 ${L4} -> xyz=0 0 ${-d2}
